File: hardware/hw_cpu/hw_cpu.kicad_pcb (KiCad board)
At the start: 2 copper layers, 89.5 x 62.2 mm, 71 parts, among them J1 CON_EXT, J2 Micro_SD_Card_Det, J3 SDIO_DEB, J4 PROG, SW1 RUN/STOP, SW2 RESTORE, SW3 DUMP, SW4 RESET, U1 STM32F429ZGTx, U2 MT48LC32M16A2P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

Commit message: Обновлена плата CPU.
Parts:
- removed C17: 4,7u 10v, Capacitors_Tantalum_SMD:CP_Tantalum_Case-A_EIA-3216-18_Reflow
Routing:
- net VREF: track 498.5 -> 495.6 mm
- net NBL0: track 21.2 -> 18.7 mm
- net VBAT: track 42.8 -> 44.8 mm
- net D4: track 23.7 -> 22.6 mm
- net D8: track 18.2 -> 18.8 mm
- net BOOT0: track 563.3 -> 562.7 mm, vias 52 -> 54
- net D9: track 17.7 -> 18.3 mm
- net SDNCAS: track 19.8 -> 20.4 mm
- net D10: track 17.5 -> 18.1 mm
Other:
- rule pad_to_mask_clearance: 0.2 -> 0.18
