File: hardware/hw_cpu/hw_cpu.kicad_pcb (KiCad board)
At the start: 2 copper layers, 89.5 x 62.2 mm, 70 parts, among them J1 CON_EXT, J2 Micro_SD_Card_Det, J3 SDIO_DEB, J4 PROG, SW1 RUN/STOP, SW2 RESTORE, SW3 DUMP, SW4 RESET, U1 STM32F429ZGTx, U2 MT48LC32M16A2P, U3 K9F5608, Y1 8MHz, Y2 32,768kHz

Commit message: Обновлены платы модулей
Other:
- net class Default: clearance 0.2 -> 0.12
- rule trace_clearance: 0.2 -> 0.12
Changed lines of the file:
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@@
-(kicad_pcb (version 20170123) (host pcbnew "(2017-06-13 revision e97f49e00)-makepkg")
+(kicad_pcb (version 4) (host pcbnew 4.0.6)
   (general
     (links 259)
     (no_connects 0)
-    (area 36.451667 64.04 160.398335 147.795001)
+    (area 36.576667 64.04 160.273334 147.795001)
     (thickness 1.6)
     (drawings 18)
@@
     (user_trace_width 0.3)
     (user_trace_width 0.5)
-    (trace_clearance 0.2)
+    (trace_clearance 0.12)
     (zone_clearance 0.25)
     (zone_45_only no)
@@
     (visible_elements 7FFFFFFF)
     (pcbplotparams
-      (layerselection 0x010f0_ffffffff)
+      (layerselection 0x010f0_80000001)
       (usegerberextensions false)
       (excludeedgelayer true)
@@
       (hpglpenspeed 20)
       (hpglpendiameter 15)
+      (hpglpenoverlay 2)
       (psnegative false)
       (psa4output false)
@@
   (net 161 "Net-(D7-Pad2)")
   (net_class Default "Это класс цепей по умолчанию."
-    (clearance 0.2)
+    (clearance 0.12)
     (trace_width 0.2)
     (via_dia 0.6)
@@
     (tags "QFP 0.5")
     (attr smd)
-    (fp_text reference U1 (at -11.735 -10.89) (layer F.SilkS)
+    (fp_text reference U1 (at -11.735 -10.89 360) (layer F.SilkS)
       (effects (font (size 1 1) (thickness 0.15)))
     )
@@
     (tags "capacitor 0805")
     (attr smd)
-    (fp_text reference C7 (at 0 -1.905) (layer F.SilkS)
+    (fp_text reference C7 (at 0 -1.905 360) (layer F.SilkS)
       (effects (font (size 1 1) (thickness 0.15)))
     )
@@
     (tags "capacitor 0402")
     (attr smd)
-    (fp_text reference C1 (at -2.54 -0.635) (layer F.SilkS)
+    (fp_text reference C1 (at -2.54 -0.635 360) (layer F.SilkS)
       (effects (font (size 1 1) (thickness 0.15)))
     )
@@
     (tags "capacitor 0402")
     (attr smd)
-    (fp_text reference C2 (at -2.54 0.635) (layer F.SilkS)
+    (fp_text reference C2 (at -2.54 0.635 360) (layer F.SilkS)
       (effects (font (size 1 1) (thickness 0.15)))
     )
@@
     (tags "capacitor 0805")
     (attr smd)
-    (fp_text reference C3 (at -2.54 0) (layer F.SilkS)
+    (fp_text reference C3 (at -2.54 0 360) (layer F.SilkS)
       (effects (font (size 1 1) (thickness 0.15)))
     )
@@
     (tags "capacitor 0402")
     (attr smd)
-    (fp_text reference C4 (at -2.0105 0) (layer F.SilkS)
+    (fp_text reference C4 (at -2.0105 0 360) (layer F.SilkS)
       (effects (font (size 1 1) (thickness 0.15)))
     )
@@
     (tags "capacitor 0402")
     (attr smd)
-    (fp_text reference C5 (at -2.625 0) (layer F.SilkS)
+    (fp_text reference C5 (at -2.625 0 360) (layer F.SilkS)
       (effects (font (size 1 1) (thickness 0.15)))
     )
@@
     (tags "capacitor 0805")
     (attr smd)
-    (fp_text reference C6 (at 0 -1.905) (layer F.SilkS)
+    (fp_text reference C6 (at 0 -1.905 360) (layer F.SilkS)
       (effects (font (size 1 1) (thickness 0.15)))
     )
@@
     (tags "capacitor 0805")
     (attr smd)
-    (fp_text reference C8 (at 0 -1.905) (layer F.SilkS)
+    (fp_text reference C8 (at 0 -1.905 360) (layer F.SilkS)
       (effects (font (size 1 1) (thickness 0.15)))
     )
@@
     (tags "capacitor 0402")
     (attr smd)
-    (fp_text reference C19 (at 1.905 0.635) (layer F.SilkS)
+    (fp_text reference C19 (at 1.905 0.635 360) (layer F.SilkS)
       (effects (font (size 1 1) (thickness 0.15)))
     )
@@
     (tags "capacitor 0805")
     (attr smd)
-    (fp_text reference C21 (at -2.54 0) (layer B.SilkS)
+    (fp_text reference C21 (at -2.54 0 360) (layer B.SilkS)
       (effects (font (size 1 1) (thickness 0.15)) (justify mirror))
     )
@@
     (tags "capacitor 0805")
     (attr smd)
-    (fp_text reference C23 (at 0 2.54) (layer B.SilkS)
+    (fp_text reference C23 (at 0 2.54 360) (layer B.SilkS)
       (effects (font (size 1 1) (thickness 0.15)) (justify mirror))
     )
@@
     (tags "capacitor 0805")
     (attr smd)
-    (fp_text reference C25 (at -2.54 0.635) (layer B.SilkS)
+    (fp_text reference C25 (at -2.54 0.635 360) (layer B.SilkS)
       (effects (font (size 1 1) (thickness 0.15)) (justify mirror))
     )
@@
     (tags "LED led 0603 SMD smd SMT smt smdled SMDLED smtled SMTLED")
     (attr smd)
-    (fp_text reference D4 (at -0.635 -1.905) (layer F.SilkS)
+    (fp_text reference D4 (at -0.635 -1.905 360) (layer F.SilkS)
       (effects (font (size 1 1) (thickness 0.15)))
     )
@@
     (tags "resistor 0805")
     (attr smd)
-    (fp_text reference R15 (at -1.27 -2.3495) (layer B.SilkS)
+    (fp_text reference R15 (at -1.27 -2.3495 360) (layer B.SilkS)
       (effects (font (size 1 1) (thickness 0.15)) (justify mirror))
     )
@@
     (tags "resistor 0805")
     (attr smd)
-    (fp_text reference R18 (at -2.54 0) (layer F.SilkS)
+    (fp_text reference R18 (at -2.54 0 360) (layer F.SilkS)
       (effects (font (size 1 1) (thickness 0.15)))
     )
@@
     (tags "resistor 0805")
     (attr smd)
-    (fp_text reference R19 (at -0.635 2.54) (layer F.SilkS)
+    (fp_text reference R19 (at -0.635 2.54 360) (layer F.SilkS)
       (effects (font (size 1 1) (thickness 0.15)))
     )

Commit message: HW: Обновлена схема CPU
Parts:
- removed J2: Micro_SD_Card_Det, w_conn_misc:Conn_uSDcard
- removed REF** (x2): MountingHole_2.2mm_M2_Pad, Mounting_Holes:MountingHole_2.2mm_M2_Pad
- removed REF** (x4): MountingHole_3.2mm_M3, Mounting_Holes:MountingHole_3.2mm_M3
- added C17: 100u, Capacitors_SMD:CP_Elec_8x6.5, F.Cu at (162.7, 128.9)
- added C27, C28, C29, C30, C31, C32, C33, C34, C38, C39, C40, C42, C43, C44, C45: 100n, Capacitors_SMD:C_0805, F.Cu at (81.0, 98.6)
- added C35: 4,7u 10v, Capacitors_Tantalum_SMD:CP_Tantalum_Case-A_EIA-3216-18_Reflow, F.Cu at (86.9, 126.4)
- added C36, C37: 2,2u, Capacitors_SMD:C_0402, F.Cu at (81.0, 98.6)
- added C41: 4,7u 10v, Capacitors_Tantalum_SMD:CP_Tantalum_Case-B_EIA-3528-21_Reflow, F.Cu at (86.1, 134.0)
- added D1: 1N5825, Diodes_SMD:D_SMA, F.Cu at (129.5, 125.1)
- added J5: TEST, Connect:he10-14d, F.Cu at (112.4, 82.4)
- added L1: 470uH, Inductors_NEOSID:Neosid_Inductor_SM-PIC1004H, F.Cu at (140.3, 123.2)
- added L2: 470uH, Inductors_NEOSID:Neosid_Inductor_SM-PIC1004H, F.Cu at (95.1, 104.0)
- added R20, R21: 1k, Resistors_SMD:R_0805, F.Cu at (81.0, 98.6)
- added R22, R23, R24, R25, R26, R27, R28: 10k, Resistors_SMD:R_0805, F.Cu at (81.0, 98.6)
- added SW5: TERMINAL, Buttons_Switches_SMD:SW_SPDT_PCM12, F.Cu at (84.0, 84.6)
- added TP1: +12V, Measurement_Points:Measurement_Point_Round-TH_Small, F.Cu at (116.8, 106.7)
- added TP2: +3,3V, Measurement_Points:Measurement_Point_Round-TH_Small, F.Cu at (152.4, 134.6)
- added TP3: RS_A, Measurement_Points:Measurement_Point_Round-TH_Small, F.Cu at (144.8, 87.6)
- added TP4: RS_B, Measurement_Points:Measurement_Point_Round-TH_Small, F.Cu at (148.6, 88.3)
- added U1: LM2596S-ADJ, TO_SOT_Packages_SMD:TO-263-5_TabPin3, F.Cu at (117.5, 126.4)
- added U2: MC34063, Housings_SOIC:SOIC-8_3.9x4.9mm_Pitch1.27mm, F.Cu at (163.2, 140.3)
- added U6: SP3485CN, Housings_SOIC:SOIC-8_3.9x4.9mm_Pitch1.27mm, F.Cu at (93.2, 88.9)
- BT1: footprint w_battery_holders:keystone_1025 -> w_battery_holders:keystone_107
- C1, C2: value 22p -> 100u; footprint Capacitors_SMD:C_0402 -> Capacitors_SMD:CP_Elec_8x6.5
- C10, C13, C14, C3, C6, C7, C8, C9: value 100n -> 100u; footprint Capacitors_SMD:C_0805 -> Capacitors_SMD:CP_Elec_8x6.5
- C16: value 100n -> 470pF; footprint Capacitors_SMD:C_0805 -> Capacitors_SMD:C_0402
- C18: value 2,2u -> 100u; footprint Capacitors_SMD:C_0402 -> Capacitors_SMD:CP_Elec_8x6.5
- C19: value 2,2u -> 22p
- C20: value 100n -> 22p; footprint Capacitors_SMD:C_0805 -> Capacitors_SMD:C_0402; moved to F.Cu
- C21: value 100n -> 12p; footprint Capacitors_SMD:C_0805 -> Capacitors_SMD:C_0402; moved to F.Cu
- C22: value 4,7u 10v -> 12p; footprint Capacitors_Tantalum_SMD:CP_Tantalum_Case-B_EIA-3528-21_Reflow -> Capacitors_SMD:C_0402
- C23, C24, C25, C26, R10, R11, R12, R13, R6, R7, R8, R9: moved to F.Cu
- C4: value 12p -> 1nF
- C5: value 12p -> 100u; footprint Capacitors_SMD:C_0402 -> Capacitors_SMD:CP_Elec_8x6.5
- D2: value PWR -> 1N5825; footprint LEDs:LED_0603 -> Diodes_SMD:D_SMA
- D3: value RUN -> PWR; footprint LEDs:LED_0603 -> LEDs:LED_0805
- D4: value STOP -> RUN; footprint LEDs:LED_0603 -> LEDs:LED_0805
- D5: value ERR -> STP; footprint LEDs:LED_0603 -> LEDs:LED_0805; moved to F.Cu
- D6, D7: footprint LEDs:LED_0603 -> LEDs:LED_0805; moved to F.Cu
- J1: value CON_EXT -> POWER; footprint Projects:Pin_Header_2.00mm_SMD -> Connectors_Phoenix:PhoenixContact_MC-G_02x3.81mm_Angled
- J3: value SDIO_DEB -> Micro_SD_Card_Det; footprint Pin_Headers:Pin_Header_Straight_1x07_Pitch2.00mm -> Projects:Conn_uSDcard
- J4: value PROG -> BUS; footprint Connect:DB9FC -> Connect:he10-10d
- R14, R15: value 10k -> 560R; moved to F.Cu
- R16: value 10k -> 120R
- R17, R18, R19: value 10k -> 1k
- R3: value 1k -> 0,3R; footprint Resistors_SMD:R_0805 -> Resistors_SMD:R_2010
- R4: value 1k -> 0,3R; footprint Resistors_SMD:R_0805 -> Resistors_SMD:R_2010; moved to F.Cu
- R5: value 1k -> 10k; moved to F.Cu
- moved BT1 104.3 mm to (178.4, 95.2), turned to 0 degrees
- moved C14 95.4 mm to (177.3, 121.9), turned to 0 degrees
- moved SW2 93.9 mm to (43.3, 146.1)
- moved C18 91.0 mm to (175.4, 135.3), turned to 0 degrees
- moved J4 84.4 mm to (153.5, 80.7), turned to 0 degrees
- moved SW1 82.1 mm to (28.4, 140.8), turned to 0 degrees
- moved J1 80.3 mm to (128.3, 148.0), turned to 0 degrees
- moved J3 75.5 mm to (47.1, 113.2), turned to 0 degrees
- moved C3 74.4 mm to (126.5, 137.8), turned to 180 degrees
- moved R3 74.2 mm to (165.8, 151.8), turned to 0 degrees
- moved C1 71.2 mm to (109.9, 150.5), turned to 180 degrees
- moved C2 70.6 mm to (138.4, 137.8), turned to 0 degrees
- moved R4 69.4 mm to (156.9, 151.8), turned to 0 degrees
- moved C13 69.4 mm to (154.4, 114.9), turned to 0 degrees
- moved R18 63.3 mm to (81.0, 98.6), turned to 0 degrees
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- renumbered U1 to U3, U2 to U4, U3 to U5
Connections:
- C1 pad 1: BOOT0 -> Net-(C1-Pad1)
- C1 pad 2: OSC_IN -> BOOT0
- C10 pad 1: VREF -> +12V
- C11 pad 1: VREF -> +12V
- C12 pad 1: VREF -> +12V
- C13 pad 1: VREF -> +12V
- C14 pad 1: VREF -> +12V
- C15 pad 1: VREF -> +12V
- C16 pad 1: VREF -> Net-(C16-Pad1)
- C18 pad 1: VCAP1 -> VREF
- C19 pad 1: VCAP2 -> BOOT0
- C19 pad 2: BOOT0 -> OSC_IN
- C2 pad 1: BOOT0 -> Net-(C1-Pad1)
- C2 pad 2: OSC_OUT -> BOOT0
- C20 pad 1: VREF -> BOOT0
- C20 pad 2: BOOT0 -> OSC_OUT
- C21 pad 1: VREF -> BOOT0
- C21 pad 2: BOOT0 -> OSC32_IN
- C22 pad 1: VREF -> BOOT0
- C22 pad 2: BOOT0 -> OSC32_OUT
- C23 pad 1: VREF -> RESET
- C26 pad 1: Net-(C26-Pad1) -> VREF
- C3 pad 1: RESET -> Net-(C1-Pad1)
- C4 pad 1: BOOT0 -> Net-(C4-Pad1)
- C4 pad 2: OSC32_IN -> +12V
- C5 pad 1: BOOT0 -> +12V
- C5 pad 2: OSC32_OUT -> BOOT0
- C6 pad 1: VREF -> +12V
- C7 pad 1: VREF -> +12V
- C8 pad 1: VREF -> +12V
- C9 pad 1: VREF -> +12V
- D2 pad 1: BOOT0 -> Net-(D2-Pad1)
- D2 pad 2: Net-(D2-Pad2) -> BOOT0
- D4 pad 1: Net-(D3-Pad2) -> BOOT0
- D4 pad 2: VREF -> Net-(D4-Pad2)
- J1 pad 1: RESET -> BOOT0
- J1 pad 2: RESET -> Net-(C1-Pad1)
- J3 pad 4: SDIO_CK -> VREF
- J3 pad 5: SDIO_D0 -> SDIO_CK
- J3 pad 6: SDIO_D1 -> BOOT0
- J3 pad 7: BOOT0 -> SDIO_D0
- J4 pad 1: UART_RX -> Net-(J4-Pad1)
- J4 pad 2: UART_TX -> Net-(J4-Pad2)
- J4 pad 4: Net-(J4-Pad4) -> BOOT0
- J4 pad 5: VREF -> BOOT0
- J4 pad 7: RESET -> +12V
- J4 pad 8: SWCLK -> +12V
- J4 pad 9: SWDIO -> +12V
- R1 pad 1: VREF -> +12V
- R1 pad 2: RESET -> Net-(C4-Pad1)
- R10 pad 1: SDIO_D2 -> VREF
- R10 pad 2: VREF -> FW_REST
- R11 pad 1: SDIO_D3 -> VREF
- R11 pad 2: VREF -> FW_DUMP
- R12 pad 1: SDIO_CMD -> NE1
- R13 pad 1: SDIO_CK -> VREF
- R13 pad 2: VREF -> Net-(C44-Pad1)
- R14 pad 1: CARD_DET -> VREF
- R14 pad 2: VREF -> Net-(J4-Pad1)
- R15 pad 1: VREF -> Net-(J4-Pad2)
- R15 pad 2: Net-(C26-Pad1) -> BOOT0
- R16 pad 1: VREF -> Net-(R16-Pad1)
- R16 pad 2: RUN -> Net-(J4-Pad2)
- R17 pad 1: VREF -> Net-(D3-Pad2)
- R17 pad 2: STOP -> LED1
- R18 pad 1: VREF -> Net-(D4-Pad2)
- R18 pad 2: FW_REST -> LED2
- R19 pad 1: VREF -> Net-(D5-Pad2)
- R19 pad 2: FW_DUMP -> LED3
- R2 pad 1: Net-(D2-Pad2) -> Net-(C4-Pad1)
- R2 pad 2: LED1 -> BOOT0
- R3 pad 1: Net-(D3-Pad2) -> Net-(R3-Pad1)
- R3 pad 2: LED2 -> +12V
- R4 pad 1: Net-(D5-Pad2) -> Net-(R3-Pad1)
- R4 pad 2: LED3 -> +12V
- R5 pad 1: Net-(D6-Pad2) -> Net-(R5-Pad1)
- R5 pad 2: LED4 -> BOOT0
- R6 pad 1: Net-(D7-Pad2) -> VREF
- R6 pad 2: LED5 -> Net-(R5-Pad1)
- R7 pad 1: NE1 -> VREF
- R7 pad 2: VREF -> RESET
- R8 pad 1: SDIO_D0 -> VREF
- R8 pad 2: VREF -> RUN
- R9 pad 1: SDIO_D1 -> VREF
- R9 pad 2: VREF -> STOP
- U3 pad 126: SPI6_SEL -> Net-(U3-Pad126)
- U3 pad 127: SPI6_MISO -> Net-(U3-Pad127)
- U3 pad 128: SPI6_SCK -> Net-(U3-Pad128)
- U3 pad 129: SPI6_MOSI -> Net-(U3-Pad129)
- U3 pad 18: SPI_SEL -> Net-(U3-Pad18)
- U3 pad 19: SPI_SCK -> Net-(U3-Pad19)
- U3 pad 20: SPI_MISO -> Net-(U3-Pad20)
- U3 pad 21: SPI_MOSI -> Net-(U3-Pad21)
- U5 pad 19: Net-(C26-Pad1) -> Net-(C44-Pad1)
Routing:
- net BOOT0: track 562.7 -> 0.00 mm, vias 54 -> 0
- net VREF: track 495.6 -> 0.00 mm, vias 25 -> 0
- net RESET: track 147.4 -> 0.00 mm, vias 2 -> 0
- net STOP: track 103.9 -> 0.00 mm, vias 2 -> 0
- net RUN: track 64.7 -> 0.00 mm
- net FW_DUMP: track 64.0 -> 0.00 mm
- net FW_REST: track 55.9 -> 0.00 mm
- net SWCLK: track 52.0 -> 0.00 mm, vias 2 -> 0
- net SWDIO: track 52.0 -> 0.00 mm, vias 2 -> 0
- net SPI6_MISO: track 48.3 -> 0.00 mm, vias 1 -> 0
- net SPI6_MOSI: track 47.6 -> 0.00 mm, vias 1 -> 0
- net SPI6_SEL: track 46.0 -> 0.00 mm, vias 1 -> 0
- net SPI6_SCK: track 46.0 -> 0.00 mm, vias 1 -> 0
- net VBAT: track 44.8 -> 0.00 mm, vias 1 -> 0
- net SDIO_D1: track 41.6 -> 0.00 mm
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- removed copper zone on B.Cu, net BOOT0
- removed copper zone on F.Cu, net BOOT0
Other:
- board outline removed
