File: hardware/hw_cpu/hw_cpu.sch (KiCad schematic (older format))
At the start: 57 parts, among them IC1 MT48LC4M16A2P, SW1 RESET, U2 STM32F429ZGTx, Y1 8MHz, Y2 32,768kHz

Commit message: Обновлена схема CPU
Parts:
- removed J?: COM_EXP, symbol CONN_01X09
- removed J?: IO_EXP, symbol CONN_01X09
- added J1: CON_EXT, Projects:Pin_Header_2.00mm_SMD, symbol CONN_02X14
- added J4: DEBUG, Pin_Headers:Pin_Header_Straight_1x07_Pitch2.00mm, symbol CONN_01X07
- BT1: footprint Connect:CR2032H -> w_battery_holders:keystone_1025
- J2: renamed from J?; footprint (none) -> Projects:Conn_uSDcard
- J3: renamed from J?; footprint (none) -> Pin_Headers:Pin_Header_Straight_1x07_Pitch2.00mm
- gave numbers to parts that had none: 1
- renumbered C14 to C10, C15 to C11, C16 to C12, C17 to C13, C18 to C14, C19 to C15, C20 to C16, C21 to C17, C22 to C18, C23 to C19, C7 to C20, C8 to C21, C9 to C22, C25 to C23, C26 to C24, C4 to C25, C24 to C26, C5 to C4, C6 to C5, C10 to C6, C11 to C7, C12 to C8, C13 to C9, R14 to R15, U2 to U1, IC1 to U2, ??1 to U3
Other:
- moved on the sheet: C20, C21, C22, C23, C24, C26, R15, R7, U2, U3

Commit message: Обновлена плата CPU
Parts:
- removed J4: DEBUG, Pin_Headers:Pin_Header_Straight_1x07_Pitch2.00mm, symbol CONN_01X07
- added J4: PROG, Connect:DB9MD, symbol DB9_FEMALE_MountingHoles
- BT1: footprint w_battery_holders:keystone_1025 -> w_battery_holders:keystone_107
Connections:
- net RESET: now also J4.7
- net SDIO_CK: now also J3.4 (P4); no longer J3.6 (P6)
- net SDIO_CMD: now also J3.3 (P3); no longer J3.5 (P5)
- net SDIO_D0: now also J3.5 (P5); no longer J3.1 (P1)
- net SDIO_D1: now also J3.6 (P6); no longer J3.2 (P2)
- net SDIO_D2: now also J3.1 (P1); no longer J3.3 (P3)
- net SDIO_D3: now also J3.2 (P2); no longer J3.4 (P4)
- net SWCLK: now also J4.8
- net SWDIO: now also J4.9
- net UART_RX: now also J4.1
- net UART_TX: now also J4.2
- net VDD: now also J4.5
- net VSS: now also J4.0 (PAD), J4.3, J4.6
Changed lines of the file:
@@
 LIBS:powerint
 LIBS:hw_cpu-cache
-EELAYER 25 0
+EELAYER 26 0
 EELAYER END
 $Descr A3 16535 11693
@@
 F 0 "BT1" H 4000 10250 50  0000 L CNN
 F 1 "Battery" H 4000 10150 50  0000 L CNN
-F 2 "w_battery_holders:keystone_1025" V 3900 10240 50  0001 C CNN
+F 2 "w_battery_holders:keystone_107" V 3900 10240 50  0001 C CNN
 F 3 "" V 3900 10240 50  0000 C CNN
 	1    3900 10200
@@
 	1    0    0    -1
 $EndComp
+Text GLabel 15300 8675 0    60   Input ~ 0
+SDIO_D2
+Text GLabel 15300 8775 0    60   Input ~ 0
+SDIO_D3
 Text GLabel 15300 8875 0    60   Input ~ 0
-SDIO_D2
+SDIO_CMD
 Text GLabel 15300 8975 0    60   Input ~ 0
-SDIO_D3
+SDIO_CK
 Text GLabel 15300 9075 0    60   Input ~ 0
-SDIO_CMD
+SDIO_D0
 Text GLabel 15300 9175 0    60   Input ~ 0
-SDIO_CK
-Text GLabel 15300 8675 0    60   Input ~ 0
-SDIO_D0
-Text GLabel 15300 8775 0    60   Input ~ 0
 SDIO_D1
 $Comp
@@
 	-1   0    0    -1
 $EndComp
-$Comp
-L CONN_01X07 J4
-U 1 1 598BFB5B
-P 9400 9100
-F 0 "J4" H 9400 9500 50  0000 C CNN
-F 1 "DEBUG" V 9500 9100 50  0000 C CNN
-F 2 "Pin_Headers:Pin_Header_Straight_1x07_Pitch2.00mm" H 9400 9100 50  0001 C CNN
-F 3 "" H 9400 9100 50  0001 C CNN
-	1    9400 9100
-	1    0    0    -1
-$EndComp
-Text GLabel 9200 8800 0    60   Input ~ 0
+Text GLabel 9175 9575 0    60   Input ~ 0
 SWDIO
-Text GLabel 9200 8900 0    60   Input ~ 0
+Text GLabel 9175 9375 0    60   Input ~ 0
 SWCLK
 $Comp
 L VDD #PWR050
 U 1 1 598C121E
-P 9200 9100
-F 0 "#PWR050" H 9200 9200 30  0001 C CNN
-F 1 "VDD" H 9200 9210 30  0000 C CNN
-F 2 "" H 9200 9100 60  0000 C CNN
-F 3 "" H 9200 9100 60  0000 C CNN
-	1    9200 9100
+P 9175 9675
+F 0 "#PWR050" H 9175 9775 30  0001 C CNN
+F 1 "VDD" H 9175 9785 30  0000 C CNN
+F 2 "" H 9175 9675 60  0000 C CNN
+F 3 "" H 9175 9675 60  0000 C CNN
+	1    9175 9675
 	0    -1   -1   0
 $EndComp
@@
 L VSS #PWR051
 U 1 1 598C12D4
-P 9200 9200
-F 0 "#PWR051" H 9200 9050 50  0001 C CNN
-F 1 "VSS" H 9200 9350 50  0000 C CNN
-F 2 "" H 9200 9200 50  0000 C CNN
-F 3 "" H 9200 9200 50  0000 C CNN
-	1    9200 9200
-	0    -1   -1   0
-$EndComp
-Text GLabel 9200 9000 0    60   Input ~ 0
+P 9175 8975
+F 0 "#PWR051" H 9175 8825 50  0001 C CNN
+F 1 "VSS" H 9175 9125 50  0000 C CNN
+F 2 "" H 9175 8975 50  0000 C CNN
+F 3 "" H 9175 8975 50  0000 C CNN
+	1    9175 8975
+	0    -1   -1   0
+$EndComp
+Text GLabel 9175 9175 0    60   Input ~ 0
 RESET
-Text GLabel 9200 9300 0    60   Input ~ 0
+Text GLabel 9175 9075 0    60   Input ~ 0
 UART_TX
-Text GLabel 9200 9400 0    60   Input ~ 0
+Text GLabel 9175 8875 0    60   Input ~ 0
 UART_RX
+$Comp
+L DB9_FEMALE_MountingHoles J4
+U 1 1 598C9A18
+P 9475 9275
+F 0 "J4" H 9654 9278 50  0000 L CNN
+F 1 "PROG" H 9654 9187 50  0000 L CNN
+F 2 "Connect:DB9MD" H 9475 9275 50  0001 C CNN
+F 3 "" H 9475 9275 50  0001 C CNN
+	1    9475 9275
+	1    0    0    -1
+$EndComp
+$Comp
+L VSS #PWR052
+U 1 1 598CA874
+P 9175 9275
+F 0 "#PWR052" H 9175 9125 50  0001 C CNN
+F 1 "VSS" H 9175 9425 50  0000 C CNN
+F 2 "" H 9175 9275 50  0000 C CNN
+F 3 "" H 9175 9275 50  0000 C CNN
+	1    9175 9275
+	0    -1   -1   0
+$EndComp
+$Comp
+L VSS #PWR053
+U 1 1 598CAB4D
+P 9475 9875
+F 0 "#PWR053" H 9475 9725 50  0001 C CNN
+F 1 "VSS" H 9475 10025 50  0000 C CNN
+F 2 "" H 9475 9875 50  0000 C CNN
+F 3 "" H 9475 9875 50  0000 C CNN
+	1    9475 9875
+	-1   0    0    1
+$EndComp
 $EndSCHEMATC

Commit message: Обновлены схема и плата CPU.
Добавлены переключатель START/STOP, кнопки DUMP и RESTORE.
Parts:
- added R16, R17, R18, R19: 10k, Resistors_SMD:R_0805, symbol R_Small
- added SW1: RUN/STOP, Buttons_Switches_ThroughHole:KSA_Tactile_SPST, symbol SW_SPDT
- added SW2: RESTORE, Buttons_Switches_SMD:SW_SPST_B3U-3000P, symbol SW_PUSH_SMALL_H
- added SW4: RESET, Buttons_Switches_SMD:SW_SPST_B3U-3000P, symbol SW_PUSH_SMALL_H
- SW3: renamed from SW1; value RESET -> DUMP
Connections:
- net RESET: now also SW4.2; no longer SW3.1
- net SPI6_MISO: now also J1.6 (P6); no longer J1.4 (P4)
- net SPI6_MOSI: now also J1.4 (P4); no longer J1.6 (P6)
- net SPI6_SCK: now also J1.8 (P8); no longer J1.10 (P10)
- net SPI6_SEL: now also J1.10 (P10); no longer J1.8 (P8)
- net SPI_MISO: now also J1.5 (P5); no longer J1.3 (P3)
- net SPI_MOSI: now also J1.3 (P3); no longer J1.5 (P5)
- net SPI_SCK: now also J1.7 (P7); no longer J1.9 (P9)
- net SPI_SEL: now also J1.9 (P9); no longer J1.7 (P7)
- net VDD: now also R16.1, R17.1, R18.1, R19.1
- net VSS: now also SW1.2 (B); no longer SW3.2
- new net FW_DUMP: R19.2, SW3.2
- new net FW_REST: R18.2, SW2.2
- new net RUN: R16.2, SW1.1 (A)
- new net STOP: R17.2, SW1.3 (C), SW2.1, SW3.1, SW4.1
Other:
- moved on the sheet: J4, SW3

Commit message: Обновлена плата CPU.
Завершена предварительная трассировка
Parts:
- removed SW2: RESTORE, Buttons_Switches_SMD:SW_SPST_B3U-3000P, symbol SW_PUSH_SMALL_H
- removed SW3: DUMP, Buttons_Switches_SMD:SW_SPST_B3U-3000P, symbol SW_PUSH_SMALL_H
- removed SW4: RESET, Buttons_Switches_SMD:SW_SPST_B3U-3000P, symbol SW_PUSH_SMALL_H
- removed U2: MT48LC4M16A2P, Housings_SSOP:TSOPII-54_10.16x22.22mm-Pitch0.8mm, symbol MT48LC4M16A2P
- added D4: STOP, LEDs:LED_0603, symbol LED-RESCUE-main
- added SW2: RESTORE, Buttons_Switches_SMD:SW_SPDT_PCM12, symbol SW_SPDT
- added SW3: DUMP, Buttons_Switches_SMD:SW_SPDT_PCM12, symbol SW_SPDT
- added SW4: RESET, Buttons_Switches_SMD:SW_SPDT_PCM12, symbol SW_SPDT
- added U2: MT48LC32M16A2P, TSOPII-54, symbol MT48LC32M16A2P
- D2: value LED -> PWR
- D3: value LED -> RUN
- D5: renamed from D4; value LED -> ERR
- D6: renamed from D5; value LED -> FLT
- D7: renamed from D6; value LED -> CFL
- J4: footprint Connect:DB9MD -> Connect:DB9FC
Connections:
- net A0: now also U2.23 (A0)
- net A1: now also U2.24 (A1)
- net A10: now also U2.22 (A10)
- net A11: now also U2.35 (A11)
- net A12: now also U2.36 (A12)
- net A14: now also U2.20 (BA0)
- net A15: now also U2.21 (BA1)
- net A2: now also U2.25 (A2)
- net A3: now also U2.26 (A3)
- net A4: now also U2.29 (A4)
- net A5: now also U2.30 (A5)
- net A6: now also U2.31 (A6)
- net A7: now also U2.32 (A7)
- net A8: now also U2.33 (A8)
- net A9: now also U2.34 (A9)
- net CARD_DET: now also J2.9 (DET_B); no longer J2.10 (DET_A)
- net D0: now also U2.2 (DQ0)
- net D1: now also U2.4 (DQ1)
- net D10: now also U2.45 (DQ10)
- net D11: now also U2.47 (DQ11)
- net D12: now also U2.48 (DQ12)
- net D13: now also U2.50 (DQ13)
- net D14: now also U2.51 (DQ14)
- net D15: now also U2.53 (DQ15)
- net D2: now also U2.5 (DQ2)
- net D3: now also U2.7 (DQ3)
- net D4: now also U2.8 (DQ4)
- net D5: now also U2.10 (DQ5)
- net D6: now also U2.11 (DQ6)
- net D7: now also U2.13 (DQ7)
- net D8: now also U2.42 (DQ8)
- net D9: now also U2.44 (DQ9)
- net FW_DUMP: now also U1.133 (I2S3_CK/SPI1_SCK/SPI3_SCK/SYS_JTDO-SWO/TIM2_CH2/PB3), SW3.3 (C)
- net FW_REST: now also U1.134 (I2S3_ext_SD/SPI1_MISO/SPI3_MISO/SYS_JTRST/TIM3_CH1/PB4), SW2.3 (C)
- net NBL0: now also U2.15 (DQML)
- net NBL1: now also U2.39 (DQMH)
- net RESET: now also SW4.3 (C)
- net RUN: now also U1.124 (PG9/DAC_EXTI9/DCMI_VSYNC/FMC_NCE3/FMC_NE2/USART6_RX)
- net SDCKE0: now also U2.37 (CKE)
- net SDCLK: now also U2.38 (CLK)
- net SDNCAS: now also U2.17 (~CAS~)
- net SDNE0: now also U2.19 (~CS~)
- net SDNRAS: now also U2.18 (~RAS~)
- net SDNWE: now also U2.16 (~WE~)
- net STOP: now also U1.125 (PG10/DCMI_D2/FMC_NCE4_1/FMC_NE3/LTDC_B2/LTDC_G3), SW2.2 (B), SW3.2 (B), SW4.2 (B)
- net VDD: now also D4.2 (A), U2.1 (VDD), U2.14 (VDD), U2.27 (VDD), U2.3 (VDDQ), U2.43 (VDDQ), U2.49 (VDDQ), U2.9 (VDDQ)
- net VSS: now also J2.10 (DET_A), U2.12 (VSSQ), U2.28 (VSS), U2.41 (VSS), U2.46 (VSSQ), U2.52 (VSSQ), U2.54 (VSS), U2.6 (VSSQ); no longer J2.9 (DET_B)
- net at D3.2 (A), R3.1: now also D4.1 (K)
Other:
- moved on the sheet: D2, R18, R19, R2, R3

Commit message: HW: Обновлена схема CPU.
Parts:
- removed D4: STOP, LEDs:LED_0603, symbol LED-RESCUE-main
- removed J1: CON_EXT, Projects:Pin_Header_2.00mm_SMD, symbol CONN_02X14
- removed J3: SDIO_DEB, Pin_Headers:Pin_Header_Straight_1x07_Pitch2.00mm, symbol CONN_01X07
- added C?: 100n, Capacitors_SMD:C_0805, symbol C_Small
- added C? (x4): 100u, symbol CP
- added C?: 100n, symbol C
- added C?: 470pF, symbol C
- added D?: 1N5819, symbol D_Schottky
- added J?: BUS, symbol CONN_02X05
- added J?: TEST, symbol CONN_02X07
- added L?: 470uH, symbol L_Core_Iron
- added R? (x2): 560R, symbol R
- added R?: 120R, symbol R
- added R? (x2): 0,3R, symbol R
- added R? (x2): R, symbol R
- added U?: SP3485CN, Housings_SOIC:SOIC-8_3.9x4.9mm_Pitch1.27mm, symbol SP3485CN
- added U?: MC34063, symbol MC34063
- D5: value ERR -> STP
Connections:
- net FW_DUMP: now also J?.12 (P12)
- net FW_REST: now also J?.11 (P11)
- net LED1: now also J?.4 (P4)
- net LED2: now also J?.5 (P5)
- net LED3: now also J?.6 (P6)
- net LED4: now also J?.7 (P7)
- net LED5: now also J?.8 (P8)
- net RESET: now also J?.13 (P13)
- net RUN: now also J?.9 (P9)
- net STOP: now also J?.10 (P10)
- net VDD: now also C?.1, C?.1, C?.1, L?.2, R?.1, R?.1, U?.8 (VCC)
- net VSS: now also C?.2, C?.2, C?.2, C?.2, C?.2, C?.2, C?.2, D?.2 (A), J?.14 (P14), J?.3 (P3), J?.4 (P4), J?.5 (P5), J?.6 (P6), R?.2, R?.2, U?.4 (GND), U?.5 (GND)
- net SPI6_MISO: no longer names the net of U1.127 (PG12/FMC_NE4/LTDC_B1/LTDC_B4/SPI6_MISO/USART6_RTS)
- net SPI6_MOSI: no longer names the net of U1.129 (PG14/ETH_TXD1/FMC_A25/SPI6_MOSI/USART6_TX)
- net SPI6_SCK: no longer names the net of U1.128 (PG13/ETH_TXD0/FMC_A24/SPI6_SCK/USART6_CTS)
- net SPI6_SEL: no longer names the net of U1.126 (PG11/ADC1_EXTI11/ADC2_EXTI11/ADC3_EXTI11/DCMI_D3/ETH_TX_EN/FMC_NCE4_2/LTDC_B3)
- net SPI_MISO: no longer names the net of U1.20 (PF8/ADC3_IN6/FMC_NIOWR/SAI1_SCK_B/SPI5_MISO/TIM13_CH1)
- net SPI_MOSI: no longer names the net of U1.21 (PF9/ADC3_IN7/DAC_EXTI9/FMC_CD/SAI1_FS_B/SPI5_MOSI/TIM14_CH1)
- net SPI_SCK: no longer names the net of U1.19 (PF7/ADC3_IN5/FMC_NREG/SAI1_MCLK_B/SPI5_SCK/TIM11_CH1/UART7_TX)
- net SPI_SEL: no longer names the net of U1.18 (PF6/ADC3_IN4/FMC_NIORD/SAI1_SD_B/SPI5_NSS/TIM10_CH1/UART7_RX)
- new net: J?.1 (P1), R?.2, U?.6 (A)
- new net: J?.2 (P2), R?.1, R?.2, U?.7 (B)
- new net: R?.1, R?.1, U?.1 (SwC), U?.7 (Ipk), U?.8 (DC)
- new net: D?.1 (K), L?.1, U?.2 (SwE)
- new net: C?.1, U?.3 (TC)
- new net: R?.1, R?.2, U?.5 (Vfb)
- new net +12V: C?.1, C?.1, C?.1, J?.10 (P10), J?.7 (P7), J?.8 (P8), J?.9 (P9), R?.2, R?.2, U?.6 (Vin(VCC))
- new net RS_EN: J?.3 (P3), U?.2 (~RE~), U?.3 (DE)
- new net RS_RX: J?.2 (P2), U?.4 (DI)
- new net RS_TX: J?.1 (P1), U?.1 (RO)
Other:
- moved on the sheet: BT1, C10, C11, C12, C13, C14, C15, C16, C17, C18, C19, C20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

Commit message: HW: Обновлена схема CPU
Parts:
- removed R?: R, symbol R
- added C1, C10, C2, C3, C5, C6, C7, C8, C9: 100u, Capacitors_SMD:CP_Elec_8x6.5, symbol CP
- added C11, C12: 100n, Capacitors_SMD:C_0805, symbol C
- added C4: 1nF, Capacitors_SMD:C_0402, symbol C
- added D1: 1N5825, Diodes_SMD:D_SMA, symbol D_Schottky
- added J1: POWER, Connectors_Phoenix:PhoenixContact_MC-G_02x3.81mm_Angled, symbol Conn_01x02
- added L1: 470uH, Inductors_NEOSID:Neosid_Inductor_SM-PIC1004H, symbol L_Core_Iron
- added R1, R5: 10k, Resistors_SMD:R_0805, symbol R_Variable
- added R2: 1k, Resistors_SMD:R_0805, symbol R
- added SW5: TERMINAL, Buttons_Switches_SMD:SW_SPDT_PCM12, symbol SW_SPDT
- added TP1: +12V, Measurement_Points:Measurement_Point_Round-TH_Small, symbol TEST
- added TP2: +3,3V, Measurement_Points:Measurement_Point_Round-TH_Small, symbol TEST
- added TP3: RS_A, Measurement_Points:Measurement_Point_Round-TH_Small, symbol TEST
- added TP4: RS_B, Measurement_Points:Measurement_Point_Round-TH_Small, symbol TEST
- added U1: LM2596S-ADJ, TO_SOT_Packages_SMD:TO-263-5_TabPin3, symbol LM2596S-ADJ
- C13, C14, C17, C18: renamed from C?; footprint (none) -> Capacitors_SMD:CP_Elec_8x6.5
- C15: renamed from C?; footprint (none) -> Capacitors_SMD:C_0805
- C16: renamed from C?; footprint (none) -> Capacitors_SMD:C_0402
- D2: renamed from D?; value 1N5819 -> 1N5825; footprint (none) -> Diodes_SMD:D_SMA
- D3: renamed from D2; footprint LEDs:LED_0603 -> LEDs:LED_0805
- D4: renamed from D3; footprint LEDs:LED_0603 -> LEDs:LED_0805
- D5, D6, D7: footprint LEDs:LED_0603 -> LEDs:LED_0805
- J4: renamed from J?; footprint (none) -> Connect:he10-10d
- J5: renamed from J?; footprint (none) -> Connect:he10-14d
- L2: renamed from L?; footprint (none) -> Inductors_NEOSID:Neosid_Inductor_SM-PIC1004H
- R14, R15, R16: renamed from R?; footprint (none) -> Resistors_SMD:R_0805
- R3, R4: renamed from R?; footprint (none) -> Resistors_SMD:R_2010
- R6: renamed from R?; value R -> 1k; footprint (none) -> Resistors_SMD:R_0805
- U2: renamed from U?; footprint (none) -> Housings_SOIC:SOIC-8_3.9x4.9mm_Pitch1.27mm
- gave numbers to parts that had none: 2
- renumbered C1 to C19, C2 to C20, C4 to C21, C5 to C22, C3 to C23, C6 to C24, C7 to C25, C8 to C26, C9 to C27, C10 to C28, C11 to C29, C12 to C30, C13 to C31, C14 to C32, C15 to C33, C16 to C34, C17 to C35, C18 to C36, C19 to C37, C25 to C38, C20 to C39, C21 to C40, C22 to C41, C23 to C42, C24 to C43, C26 to C44, J4 to J2, J2 to J3, R18 to R10, R19 to R11, R7 to R12, R15 to R13, R2 to R17, R3 to R18, R4 to R19, R5 to R20, R6 to R21, R8 to R22, R9 to R23, R10 to R24, R11 to R25, R12 to R26, R13 to R27, R14 to R28, R1 to R7, R16 to R8, R17 to R9, U1 to U3, U2 to U4, U3 to U5
Connections:
- net +12V: now also C10.1, C11.1, C12.1, C4.2, C5.1, C6.1, C7.1, C8.1, C9.1, L1.2, R1.1, TP1.1
- net VDD: now also TP2.1
- net VSS: now also C1.2, C10.2, C11.2, C12.2, C2.2, C3.2, C5.2, C6.2, C7.2, C8.2, C9.2, D1.2 (A), J1.1 (Pin_1), R2.2, R5.2, U1.3 (GND), U1.5 (~ON~/OFF)
- net at J4.1 (P1), R14.2, U6.6 (A): now also SW5.3 (C), TP3.1
- net at J4.2 (P2), R15.1, R16.2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: now also TP4.1
- net at R16.1: now also SW5.2 (B)
- net at R6.2, U2.5 (Vfb): now also R5.1
- new net: C1.1, C2.1, C3.1, J1.2 (Pin_2), U1.1 (VIN)
- new net: D1.1 (K), L1.1, U1.2 (OUT)
- new net: C4.1, R1.2, R2.1, U1.4 (FB)
Other:
- moved on the sheet: D3, R17
