File: hardware/hw_cross/cross.kicad_pcb (KiCad board)
At the start: 2 copper layers, 87 x 95.9 mm, 45 parts, among them J1 MOD_IN, J2 MOD_OUT

Commit message: Обновлена плата кросс-модуля.
Добавлена буферизация шины.
Parts:
- added U1: 74LS125, Housings_SOIC:SOIC-14_3.9x8.7mm_Pitch1.27mm, B.Cu at (208.6, 179.8)
- added U1: 74LS125, Housings_SOIC:SOIC-14_3.9x8.7mm_Pitch1.27mm, B.Cu at (178.6, 179.8)
- added U1: 74LS125, Housings_SOIC:SOIC-14_3.9x8.7mm_Pitch1.27mm, B.Cu at (148.6, 179.8)
- added U1: 74LS125, Housings_SOIC:SOIC-14_3.9x8.7mm_Pitch1.27mm, B.Cu at (208.6, 146.8)
- added U1: 74LS125, Housings_SOIC:SOIC-14_3.9x8.7mm_Pitch1.27mm, B.Cu at (178.6, 146.8)
- added U1: 74LS125, Housings_SOIC:SOIC-14_3.9x8.7mm_Pitch1.27mm, B.Cu at (148.6, 146.8)
- added U1: 74LS125, Housings_SOIC:SOIC-14_3.9x8.7mm_Pitch1.27mm, B.Cu at (208.6, 113.8)
- added U1: 74LS125, Housings_SOIC:SOIC-14_3.9x8.7mm_Pitch1.27mm, B.Cu at (178.6, 113.8)
- added U1: 74LS125, Housings_SOIC:SOIC-14_3.9x8.7mm_Pitch1.27mm, B.Cu at (148.6, 113.8)
Connections:
- net Net-(J1-Pad5) renamed SEL
- J1 pad 1: Net-(J1-Pad1) -> RESET_IN (x9)
- J1 pad 10: Net-(J1-Pad10) -> VCC (x9)
- J1 pad 11: Net-(J1-Pad11) -> GND (x9)
- J1 pad 12: Net-(J1-Pad12) -> GND (x9)
- J1 pad 13: Net-(J1-Pad13) -> GND (x9)
- J1 pad 14: Net-(J1-Pad14) -> GND (x9)
- J1 pad 2: Net-(J1-Pad2) -> SCK_IN (x9)
- J1 pad 3: Net-(J1-Pad3) -> MISO_OUT (x9)
- J1 pad 4: Net-(J1-Pad4) -> MOSI_IN (x9)
- J1 pad 6: Net-(J1-Pad6) -> VCC (x9)
- J1 pad 7: Net-(J1-Pad7) -> VCC (x9)
- J1 pad 8: Net-(J1-Pad8) -> VCC (x9)
- J1 pad 9: Net-(J1-Pad9) -> VCC (x9)
- J2 pad 1: Net-(J1-Pad1) -> RESET_OUT (x9)
- J2 pad 10: Net-(J1-Pad10) -> VCC (x9)
- J2 pad 11: Net-(J1-Pad11) -> GND (x9)
- J2 pad 12: Net-(J1-Pad12) -> GND (x9)
- J2 pad 13: Net-(J1-Pad13) -> GND (x9)
- J2 pad 14: Net-(J1-Pad14) -> GND (x9)
- J2 pad 2: Net-(J1-Pad2) -> SCK_OUT (x9)
- J2 pad 3: Net-(J1-Pad3) -> MISO_IN (x9)
- J2 pad 4: Net-(J1-Pad4) -> MOSI_OUT (x9)
- J2 pad 6: Net-(J1-Pad6) -> VCC (x9)
- J2 pad 7: Net-(J1-Pad7) -> VCC (x9)
- J2 pad 8: Net-(J1-Pad8) -> VCC (x9)
- J2 pad 9: Net-(J1-Pad9) -> VCC (x9)
Routing:
- net Net-(J1-Pad13): track 438.0 -> 0.00 mm
- net Net-(J1-Pad2): track 436.6 -> 0.00 mm
- net Net-(J1-Pad3): track 423.8 -> 0.00 mm
- net Net-(J1-Pad12): track 423.3 -> 0.00 mm
- net Net-(J1-Pad14): track 420.5 -> 0.00 mm
- net Net-(J1-Pad1): track 419.1 -> 0.00 mm
- net SEL: track 411.5 -> 0.00 mm
- net Net-(J1-Pad9): track 411.5 -> 0.00 mm
- net Net-(J1-Pad8): track 411.5 -> 0.00 mm
- net Net-(J1-Pad7): track 411.5 -> 0.00 mm
- net Net-(J1-Pad6): track 411.5 -> 0.00 mm
- net Net-(J1-Pad4): track 411.5 -> 0.00 mm
- net Net-(J1-Pad11): track 411.5 -> 0.00 mm
- net Net-(J1-Pad10): track 411.5 -> 0.00 mm
- net GND: track 0.00 -> 330.2 mm, vias 0 -> 45
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- added copper zone on F.Cu, net GND
- added copper zone on F.Cu, net VCC
